Commit message: add drone visualization in rviz

File: src/px4_rotor_sim/model/iris.urdf (robot description, URDF)
Before this commit: robot iris, 7 links, 6 joints
Links:
- removed link iris__/imu_link
- removed link iris__base_link
- removed link iris__gps0__link
- removed link iris__rotor_0
- removed link iris__rotor_1
- removed link iris__rotor_2
- removed link iris__rotor_3
- added link base_link, mass 1.5; collision box size=0.47 0.47 0.11; visual mesh filename=package://px4_rotor_sim/model/meshes/iris.stl scale=1 1 1
- added link gps0__link, mass 0.015; visual cylinder length=0.002 radius=0.01
- added link imu_link, mass 0.015
- added link rotor_0, mass 0.005; collision cylinder length=0.005 radius=0.128; visual mesh filename=package://px4_rotor_sim/model/meshes/iris_prop_ccw.dae scale=1 1 1
- added link rotor_1, mass 0.005; collision cylinder length=0.005 radius=0.128; visual mesh filename=package://px4_rotor_sim/model/meshes/iris_prop_ccw.dae scale=1 1 1
- added link rotor_2, mass 0.005; collision cylinder length=0.005 radius=0.128; visual mesh filename=package://px4_rotor_sim/model/meshes/iris_prop_cw.dae scale=1 1 1
- added link rotor_3, mass 0.005; collision cylinder length=0.005 radius=0.128; visual mesh filename=package://px4_rotor_sim/model/meshes/iris_prop_cw.dae scale=1 1 1
Joints:
- removed joint iris__/imu_joint
- removed joint iris__gps0_joint
- removed joint iris__rotor_0_joint
- removed joint iris__rotor_1_joint
- removed joint iris__rotor_2_joint
- removed joint iris__rotor_3_joint
- added joint gps0_joint: type fixed, parent base_link, child gps0__link, origin xyz=0.1 0  0 rpy=0 0 0, axis 0 0 0, limit lower=0 upper=0 effort=0 velocity=0
- added joint imu_joint: type fixed, parent base_link, child imu_link, origin xyz=0 0 0 rpy=0 0 0, axis 1 0 0, limit lower=0.0 upper=0.0 effort=0.0 velocity=0.0
- added joint rotor_0_joint: type revolute, parent base_link, child rotor_0, origin xyz=0.13  -0.22   0.023 rpy=0 0 0, axis 0 0 1, limit lower=-1e+16 upper=1e+16 effort=0.0 velocity=0.0
- added joint rotor_1_joint: type revolute, parent base_link, child rotor_1, origin xyz=-0.13   0.2    0.023 rpy=0 0 0, axis 0 0 1, limit lower=-1e+16 upper=1e+16 effort=0.0 velocity=0.0
- added joint rotor_2_joint: type revolute, parent base_link, child rotor_2, origin xyz=0.13  0.22  0.023 rpy=0 0 0, axis 0 0 1, limit lower=-1e+16 upper=1e+16 effort=0.0 velocity=0.0
- added joint rotor_3_joint: type revolute, parent base_link, child rotor_3, origin xyz=-0.13  -0.2    0.023 rpy=0 0 0, axis 0 0 1, limit lower=-1e+16 upper=1e+16 effort=0.0 velocity=0.0

Commit message: add path visualization

File: src/px4_rotor_sim/model/iris.urdf (robot description, URDF)
Before this commit: robot iris, 7 links, 6 joints
Links:
- link base_link: mass 1.5 -> None
- link gps0__link: geometry 
- link rotor_0: geometry collision cylinder length=0.005 radius=0.128; visual mesh filename=package://px4_rotor_sim/model/meshes/iris_prop_ccw.stl scale=1 1 1
- link rotor_1: geometry collision cylinder length=0.005 radius=0.128; visual mesh filename=package://px4_rotor_sim/model/meshes/iris_prop_ccw.stl scale=1 1 1
- link rotor_2: geometry collision cylinder length=0.005 radius=0.128; visual mesh filename=package://px4_rotor_sim/model/meshes/iris_prop_cw.stl scale=1 1 1
- link rotor_3: geometry collision cylinder length=0.005 radius=0.128; visual mesh filename=package://px4_rotor_sim/model/meshes/iris_prop_cw.stl scale=1 1 1
