Commit message: add tello visualization

File: src/tello_sim/model/tello.urdf (robot description, URDF)
Before this commit: robot iris, 7 links, 6 joints
Links:
- removed link gps0__link
- removed link imu_link
- link base_link: geometry collision box size=0.10 0.04 0.03; visual mesh filename=package://tello_sim/model/meshes/tello_body.dae scale=1 1 1
- link rotor_0: geometry collision cylinder length=0.005 radius=0.04; visual mesh filename=package://tello_sim/model/meshes/tello_prop_ccw.stl scale=1 1 1
- link rotor_1: geometry collision cylinder length=0.005 radius=0.04; visual mesh filename=package://tello_sim/model/meshes/tello_prop_ccw.stl scale=1 1 1
- link rotor_2: geometry collision cylinder length=0.005 radius=0.04; visual mesh filename=package://tello_sim/model/meshes/tello_prop_cw.stl scale=1 1 1
- link rotor_3: geometry collision cylinder length=0.005 radius=0.04; visual mesh filename=package://tello_sim/model/meshes/tello_prop_cw.stl scale=1 1 1
Joints:
- removed joint gps0_joint
- removed joint imu_joint
- joint rotor_0_joint: origin xyz=0.13  -0.22   0.023 rpy=0 0 0 -> xyz=0.0628  -0.0698   0.013 rpy=0 0 0
- joint rotor_1_joint: origin xyz=-0.13   0.2    0.023 rpy=0 0 0 -> xyz=-0.0698   0.0705    0.013 rpy=0 0 0
- joint rotor_2_joint: origin xyz=0.13  0.22  0.023 rpy=0 0 0 -> xyz=0.0628  0.0698  0.013 rpy=0 0 0
- joint rotor_3_joint: origin xyz=-0.13  -0.2    0.023 rpy=0 0 0 -> xyz=-0.0688  -0.0698   0.013 rpy=0 0 0
