Commit message: separate fw_plane_sim

File: src/fw_plane_sim/model/plane.urdf (robot description, URDF)
Before this commit: robot plane, 10 links, 9 joints
Links:
- link base_link: geometry collision box size=0.47 0.47 0.11; visual mesh filename=package://fw_plane_sim/model/meshes/body.dae scale=1 1 1
- link elevator: geometry visual mesh filename=package://fw_plane_sim/model/meshes/elevators.dae scale=1 1 1
- link left_elevon: geometry visual mesh filename=package://fw_plane_sim/model/meshes/left_aileron.dae scale=1 1 1
- link left_flap: geometry visual mesh filename=package://fw_plane_sim/model/meshes/left_flap.dae scale=1 1 1
- link right_elevon: geometry visual mesh filename=package://fw_plane_sim/model/meshes/right_aileron.dae scale=1 1 1
- link right_flap: geometry visual mesh filename=package://fw_plane_sim/model/meshes/right_flap.dae scale=1 1 1
- link rotor_puller: geometry collision cylinder length=0.005 radius=0.1; visual mesh filename=package://fw_plane_sim/model/meshes/iris_prop_ccw.dae scale=10 10 10
- link rudder: geometry visual mesh filename=package://fw_plane_sim/model/meshes/rudder.dae scale=1 1 1
Joints:
- joint rotor_puller_joint: origin xyz=0.3   0    0.246 rpy=0   1.57 0 -> xyz=1.57   0    1.0 rpy=0   1.57 0

Commit message: change fixed wing model color to red

File: src/fw_plane_sim/model/plane.urdf (robot description, URDF)
Before this commit: robot plane, 10 links, 9 joints
Links:
- link base_link: geometry collision box size=0.47 0.47 0.11; visual mesh filename=package://fw_plane_sim/model/meshes/body.stl scale=0.025 0.025 0.025
- link elevator: geometry visual mesh filename=package://fw_plane_sim/model/meshes/elevators.stl scale=0.025 0.025 0.025
- link left_elevon: geometry visual mesh filename=package://fw_plane_sim/model/meshes/left_aileron.stl scale=0.025 0.025 0.025
- link left_flap: geometry visual mesh filename=package://fw_plane_sim/model/meshes/left_flap.stl scale=0.025 0.025 0.025
- link right_elevon: geometry visual mesh filename=package://fw_plane_sim/model/meshes/right_aileron.stl scale=0.025 0.025 0.025
- link right_flap: geometry visual mesh filename=package://fw_plane_sim/model/meshes/right_flap.stl scale=0.025 0.025 0.025
- link rotor_puller: geometry collision cylinder length=0.005 radius=0.1; visual mesh filename=package://fw_plane_sim/model/meshes/iris_prop_ccw.stl scale=10 10 10
- link rudder: geometry visual mesh filename=package://fw_plane_sim/model/meshes/rudder.stl scale=0.025 0.025 0.025
